File: schematics/spinnaker_kicad/spinnaker.kicad_pcb (KiCad board)
At the start: 2 copper layers, 87 x 60.3 mm, 156 parts, among them J1 L_INP, J2 R_INP, J3 L_OUT, J4 R_OUT, J5 9VDC POWER, J6 CONTROL, Q1 AO3401, U1 SpinSemi_FV-1, U10 24LC32, U11 24LC32, U12 24LC32, U13 24LC32, U14 24LC32, U15 24LC32, U16 24LC32, U17 AMS1117-3.3, U18 AMS1117-5.0, U19 MP1470, U2 TL071, U3 TL071, U4 TL071, U5 TL071, U6 PT2258, U7 MCP4728, U8 PCF8574, U9 24LC32, Y1 32768Hz

Commit message: Files upgraded to KICAD_v9.
Other:
- net class Default removed
